Commit message: checkin testing, still broken

File: description/stretch_re3_cartesian.urdf (robot description, URDF)
Before this commit: robot stretch_full, 20 links, 19 joints
Links:
- removed link z_virtual_link
- added link x_virtual_link, mass 1.0
Joints:
- removed joint z_revolute_joint
- added joint x_prismatic_joint: type prismatic, parent virtual_base_link, child x_virtual_link, origin xyz=0.0 0.0 0.0 rpy=0.0 -0.0 0.0, axis 1. 0. 0., limit lower=-100.0 upper=100.0 effort=10.0 velocity=1.0
- joint virtual_base_joint: parent z_virtual_link -> x_virtual_link
